File: V2.kicad_pcb (KiCad board)
At the start: 4 copper layers, 58 x 49 mm, 48 parts, among them J1 MOL Pico 4, J2 MOL Pico 4, J3 MOL Pico 4, J4 MOL Pico 2, Q1 IPZ40N04S5-3R1, Q2 IPZ40N04S5-3R1, U1 PTPS55288RPMR, U2 AD5258BRMZ1, U3 C1T 4

Commit message: V2: Faulty Second Version
Parts:
- Cdith1: renamed from Cdith1 ->
- L1: footprint Cryocooler_footprints:XAL8080-103MED -> Cryocooler_footprints:XAL1010
- Rfsw1: renamed from Rfsw1 ->
- TP_AGND1: renamed from AGND; footprint TestPoint:TestPoint_Pad_D1.5mm -> TestPoint:TestPoint_THTPad_D1.5mm_Drill0.7mm
- TP_PGND1: renamed from PGND; footprint TestPoint:TestPoint_Pad_D1.5mm -> TestPoint:TestPoint_THTPad_D1.5mm_Drill0.7mm
- TP_SCL1: renamed from SCL; footprint TestPoint:TestPoint_Pad_D1.5mm -> TestPoint:TestPoint_THTPad_D1.5mm_Drill0.7mm
- TP_SDA1: renamed from SDA; footprint TestPoint:TestPoint_Pad_D1.5mm -> TestPoint:TestPoint_THTPad_D1.5mm_Drill0.7mm
- TP_VIN1: renamed from VIN; footprint TestPoint:TestPoint_Pad_D1.5mm -> TestPoint:TestPoint_THTPad_D1.5mm_Drill0.7mm
- TP_VOUT1: renamed from VOUT; footprint TestPoint:TestPoint_Pad_D1.5mm -> TestPoint:TestPoint_THTPad_D1.5mm_Drill0.7mm
- moved TP_VIN1 0.80 mm to (123.3, 91.4)
- moved L1 0.18 mm to (135.2, 87.6)
- renumbered CVCC-> to CVCC1
Connections:
- net VIN_pre renamed VIN_PRE
- U1 pad 11: Net-(U1-ISP) -> (no net)
- U1 pad 21: Net-(U1-SW2) -> (no net)
- U1 pad 9: PGND -> (no net)
Routing:
- net CRYO_2: track 44.9 -> 48.1 mm
- net CRYO_1: track 55.7 -> 58.8 mm
- net Net-(U1-SW1): track 16.9 -> 18.5 mm
Other:
- board text added: "AGND"
- board text added: "Cryocooler Board V2 Rodrigo Spinola e Castro"
- board text added: "PGND"
- board text added: "SCL"
- board text added: "SDA"
- board text added: "VIN"
- board text added: "VOUT"
- board text removed: "Cryocooler Board V1 Rodrigo Spinola e Castro"
