File: V2.kicad_sch (KiCad schematic)
At the start: 48 parts, among them J1 MOL Pico 4, J2 MOL Pico 4, J3 MOL Pico 4, J4 MOL Pico 2, Q1 IPZ40N04S5-3R1, Q2 IPZ40N04S5-3R1, U1 PTPS55288RPMR, U2 AD5258BRMZ1, U3 C1T 4

Commit message: V2: Faulty Second Version
Parts:
- L1: footprint Cryocooler_footprints:XAL8080-103MED -> Cryocooler_footprints:XAL1010
- TP_AGND1: renamed from TP5; footprint TestPoint:TestPoint_Pad_D1.5mm -> TestPoint:TestPoint_THTPad_D1.5mm_Drill0.7mm
- TP_PGND1: renamed from TP6; footprint TestPoint:TestPoint_Pad_D1.5mm -> TestPoint:TestPoint_THTPad_D1.5mm_Drill0.7mm
- TP_SCL1: renamed from TP3; footprint TestPoint:TestPoint_Pad_D1.5mm -> TestPoint:TestPoint_THTPad_D1.5mm_Drill0.7mm
- TP_SDA1: renamed from TP4; footprint TestPoint:TestPoint_Pad_D1.5mm -> TestPoint:TestPoint_THTPad_D1.5mm_Drill0.7mm
- TP_VIN1: renamed from TP2; footprint TestPoint:TestPoint_Pad_D1.5mm -> TestPoint:TestPoint_THTPad_D1.5mm_Drill0.7mm
- TP_VOUT1: renamed from TP1; footprint TestPoint:TestPoint_Pad_D1.5mm -> TestPoint:TestPoint_THTPad_D1.5mm_Drill0.7mm
Connections:
- net VIN: no longer J1.1, J1.2, U3.1
- new net VIN_PRE: J1.1, J1.2, U3.1
Changed lines of the file:
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@@
 	(wire
 		(pts
-			(xy 20.32 80.01) (xy 22.86 80.01)
-		)
-		(stroke
-			(width 0)
-			(type default)
-		)
-	)
-	(wire
-		(pts
 			(xy 109.22 49.53) (xy 109.22 54.61)
 		)
@@
 	(wire
 		(pts
+			(xy 40.64 76.2) (xy 40.64 80.01)
+		)
+		(stroke
+			(width 0)
+			(type default)
+		)
+	)
+	(wire
+		(pts
 			(xy 100.33 152.4) (xy 100.33 147.32)
 		)
@@
 	(wire
 		(pts
+			(xy 22.86 76.2) (xy 22.86 80.01)
+		)
+		(stroke
+			(width 0)
+			(type default)
+		)
+	)
+	(wire
+		(pts
 			(xy 22.86 158.75) (xy 22.86 153.67)
 		)
@@
 		)
 	)
+	(global_label "VIN"
+		(shape input)
+		(at 40.64 76.2 90)
+		(fields_autoplaced yes)
+		(effects
+			(font
+				(size 1.27 1.27)
+			)
+			(justify left)
+		)
+		(property "Intersheetrefs" "${INTERSHEET_REFS}"
+			(at 40.64 70.1909 90)
+			(effects
+				(font
+					(size 1.27 1.27)
+				)
+				(justify left)
+				(hide yes)
+			)
+		)
+	)
 	(global_label "SDA"
 		(shape input)
@@
 		)
 	)
-	(global_label "VIN"
+	(global_label "VIN_PRE"
 		(shape input)
-		(at 20.32 80.01 180)
+		(at 22.86 76.2 90)
 		(fields_autoplaced yes)
 		(effects
@@
 				(size 1.27 1.27)
 			)
-			(justify right)
+			(justify left)
 		)
 		(property "Intersheetrefs" "${INTERSHEET_REFS}"
-			(at 14.3109 80.01 0)
+			(at 22.86 65.5343 90)
 			(effects
 				(font
 					(size 1.27 1.27)
 				)
-				(justify right)
+				(justify left)
 				(hide yes)
 			)
@@
 		)
 	)
-	(global_label "VIN"
+	(global_label "VIN_PRE"
 		(shape input)
 		(at 30.48 149.86 90)
@@
 		)
 		(property "Intersheetrefs" "${INTERSHEET_REFS}"
-			(at 30.48 143.8509 90)
+			(at 30.48 139.1943 90)
 			(effects
 				(font
@@
 		(on_board yes)
 		(dnp no)
-		(property "Reference" "TP5"
+		(property "Reference" "TP_AGND1"
 			(at 78.74 154.686 90)
 			(effects
@@
 				)
 				(justify right)
+				(hide yes)
 			)
 		)
-		(property "Footprint" "TestPoint:TestPoint_Pad_D1.5mm"
+		(property "Footprint" "TestPoint:TestPoint_THTPad_D1.5mm_Drill0.7mm"
 			(at 85.09 152.4 0)
 			(effects
@@
 			(project "try_1_tps5288"
 				(path "/fc4eef0c-f0fe-4c26-9eed-35cfade9960a"
-					(reference "TP5")
+					(reference "TP_AGND1")
 					(unit 1)
 				)
@@
 		(on_board yes)
 		(dnp no)
-		(property "Reference" "TP1"
+		(property "Reference" "TP_VOUT1"
 			(at 272.034 71.12 0)
 			(effects
@@
 			)
 		)
-		(property "Footprint" "TestPoint:TestPoint_Pad_D1.5mm"
+		(property "Footprint" "TestPoint:TestPoint_THTPad_D1.5mm_Drill0.7mm"
 			(at 274.32 77.47 0)
 			(effects
@@
 			(project "try_1_tps5288"
 				(path "/fc4eef0c-f0fe-4c26-9eed-35cfade9960a"
-					(reference "TP1")
+					(reference "TP_VOUT1")
 					(unit 1)
 				)
@@
 		(on_board yes)
 		(dnp no)
-		(property "Reference" "TP3"
+		(property "Reference" "TP_SCL1"
 			(at 101.092 161.798 0)
 			(effects
@@
 				)
 				(justify right)
+				(hide yes)
 			)
 		)
-		(property "Footprint" "TestPoint:TestPoint_Pad_D1.5mm"
+		(property "Footprint" "TestPoint:TestPoint_THTPad_D1.5mm_Drill0.7mm"
 			(at 107.95 165.1 0)
 			(effects
@@
 			(project "try_1_tps5288"
 				(path "/fc4eef0c-f0fe-4c26-9eed-35cfade9960a"
-					(reference "TP3")
+					(reference "TP_SCL1")
 					(unit 1)
 				)
@@
 		(on_board yes)
 		(dnp no)
-		(property "Reference" "TP2"
+		(property "Reference" "TP_VIN1"
 			(at 38.354 73.66 0)
 			(effects
@@
 				)
 				(justify right)
+				(hide yes)
 			)
 		)
-		(property "Footprint" "TestPoint:TestPoint_Pad_D1.5mm"
+		(property "Footprint" "TestPoint:TestPoint_THTPad_D1.5mm_Drill0.7mm"
 			(at 40.64 80.01 0)
 			(effects
@@
 			(project ""
 				(path "/fc4eef0c-f0fe-4c26-9eed-35cfade9960a"
-					(reference "TP2")
+					(reference "TP_VIN1")
 					(unit 1)
 				)
@@
 			)
 		)
-		(property "Footprint" "Cryocooler_footprints:XAL8080-103MED"
+		(property "Footprint" "Cryocooler_footprints:XAL1010"
 			(at 158.75 49.53 0)
 			(effects
@@
 		(on_board yes)
 		(dnp no)
-		(property "Reference" "TP4"
+		(property "Reference" "TP_SDA1"
 			(at 101.092 173.99 0)
 			(effects
@@
 				)
 				(justify right)
+				(hide yes)
 			)
 		)
-		(property "Footprint" "TestPoint:TestPoint_Pad_D1.5mm"
+		(property "Footprint" "TestPoint:TestPoint_THTPad_D1.5mm_Drill0.7mm"
 			(at 97.79 167.64 0)
 			(effects
@@
 			(project "try_1_tps5288"
 				(path "/fc4eef0c-f0fe-4c26-9eed-35cfade9960a"
-					(reference "TP4")
+					(reference "TP_SDA1")
 					(unit 1)
 				)
@@
 		(on_board yes)
 		(dnp no)
-		(property "Reference" "TP6"
+		(property "Reference" "TP_PGND1"
 			(at 67.31 89.916 90)
 			(effects
@@
 				)
 				(justify right)
+				(hide yes)
 			)
 		)
-		(property "Footprint" "TestPoint:TestPoint_Pad_D1.5mm"
+		(property "Footprint" "TestPoint:TestPoint_THTPad_D1.5mm_Drill0.7mm"
 			(at 73.66 87.63 0)
 			(effects
@@
 			(project "try_1_tps5288"
 				(path "/fc4eef0c-f0fe-4c26-9eed-35cfade9960a"
-					(reference "TP6")
+					(reference "TP_PGND1")
 					(unit 1)
 				)
