File: V3.kicad_pcb (KiCad board)
At the start: 4 copper layers, 58 x 49 mm, 48 parts, among them J1 MOL Pico 4, J2 MOL Pico 4, J3 MOL Pico 4, J4 MOL Pico 2, Q1 IPZ40N04S5-3R1, Q2 IPZ40N04S5-3R1, U1 PTPS55288RPMR, U2 AD5258BRMZ1, U3 C1T 4

Commit message: V3: Working third version, however, still too lossy due to imbalances
Connections:
- C1 pad 1: Net-(U1-SW2) -> Net-(C1-Pad1)
- L1 pad 2: Net-(U1-SW2) -> Net-(C1-Pad1)
- U1 pad 21: (no net) -> Net-(C1-Pad1)
- U1 pad 25: Net-(U1-SW2) -> Net-(C1-Pad1)
- U1 pad 9: (no net) -> PGND
Routing:
- added copper zone on F.Cu, net Net-(C1-Pad1)
- removed copper zone on F.Cu, net Net-(U1-SW2)
Other:
- board text added: "Cryocooler Board V3 Rodrigo Spinola e Castro"
- board text removed: "Cryocooler Board V2 Rodrigo Spinola e Castro"
