File: V3.kicad_sch (KiCad schematic)
At the start: 48 parts, among them J1 MOL Pico 4, J2 MOL Pico 4, J3 MOL Pico 4, J4 MOL Pico 2, Q1 IPZ40N04S5-3R1, Q2 IPZ40N04S5-3R1, U1 PTPS55288RPMR, U2 AD5258BRMZ1, U3 C1T 4

Commit message: V3: Working third version, however, still too lossy due to imbalances
Parts:
- L1: Check_prices https://www.snapeda.com/parts/XAL1010-472MED/Coilcraft/view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 -> https://www.coilcraft.com/en-us/products/power/shielded-ind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; DESCRIPTION 4.7 µH Shielded Molded Inductor 17.5 A 5.7mOhm Max Nonstand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 -> 10 µH Shielded Molded Inductor 17.5 A 5.7mOhm Max Nonstanda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; Description_1 4.7 µH Shielded Molded Inductor 17.5 A 5.7mOhm Max Nonstand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 -> 10 µH Shielded Molded Inductor 17.5 A 5.7mOhm Max Nonstanda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; MP XAL1010-472MED -> XAL1010-103MED; PURCHASE-URL https://pricing.snapeda.com/search/part/XAL1010-472MED/?ref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 -> https://www.coilcraft.com/en-us/products/power/shielded-ind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
Connections:
- net PGND: now also U1.9 (PGND)
- net at C1.1, L1.2, U1.25 (SW2): now also U1.21 (SW2)
Changed lines of the file:
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@@
 	)
 	(junction
+		(at 168.91 63.5)
+		(diameter 0)
+		(color 0 0 0 0)
+	)
+	(junction
 		(at 73.66 92.71)
 		(diameter 0)
@@
 	)
 	(junction
+		(at 187.96 85.09)
+		(diameter 0)
+		(color 0 0 0 0)
+	)
+	(junction
 		(at 95.25 147.32)
 		(diameter 0)
@@
 	(wire
 		(pts
+			(xy 165.1 63.5) (xy 168.91 63.5)
+		)
+		(stroke
+			(width 0)
+			(type default)
+		)
+	)
+	(wire
+		(pts
 			(xy 102.87 160.02) (xy 106.68 160.02)
 		)
@@
 	(wire
 		(pts
+			(xy 187.96 82.55) (xy 187.96 85.09)
+		)
+		(stroke
+			(width 0)
+			(type default)
+		)
+	)
+	(wire
+		(pts
 			(xy 102.87 157.48) (xy 102.87 160.02)
 		)
@@
 		(pin "20"
 		)
+		(pin "9"
+		)
+		(pin "21"
+		)
 		(instances
 			(project ""
@@
 			)
 		)
-		(property "DESCRIPTION" "4.7 µH Shielded Molded Inductor 17.5 A 5.7mOhm Max Nonstandard"
+		(property "DESCRIPTION" "10 µH Shielded Molded Inductor 17.5 A 5.7mOhm Max Nonstandard"
 			(at 158.75 49.53 0)
 			(effects
@@
 			)
 		)
-		(property "Check_prices" "https://www.snapeda.com/parts/XAL1010-472MED/Coilcraft/view-part/?ref=eda"
+		(property "Check_prices" "https://www.coilcraft.com/en-us/products/power/shielded-inductors/molded-inductor/xal/xal1010/xal1010-103/"
 			(at 158.75 49.53 0)
 			(effects
@@
 			)
 		)
-		(property "MP" "XAL1010-472MED"
+		(property "MP" "XAL1010-103MED"
 			(at 158.75 49.53 0)
 			(effects
@@
 			)
 		)
-		(property "Description_1" "\n                        \n                            4.7 µH Shielded Molded Inductor 17.5 A 5.7mOhm Max Nonstandard\n                        \n"
+		(property "Description_1" "\n                        \n                            10 µH Shielded Molded Inductor 17.5 A 5.7mOhm Max Nonstandard\n                        \n"
 			(at 158.75 49.53 0)
 			(effects
@@
 			)
 		)
-		(property "PURCHASE-URL" "https://pricing.snapeda.com/search/part/XAL1010-472MED/?ref=eda"
+		(property "PURCHASE-URL" "https://www.coilcraft.com/en-us/products/power/shielded-inductors/molded-inductor/xal/xal1010/xal1010-103/"
 			(at 158.75 49.53 0)
 			(effects
