File: V4.kicad_sch (KiCad schematic)
At the start: 48 parts, among them J1 MOL Pico 4, J2 MOL Pico 4, J3 MOL Pico 4, J4 MOL Pico 2, Q1 IPZ40N04S5-3R1, Q2 IPZ40N04S5-3R1, U1 PTPS55288RPMR, U2 AD5258BRMZ1, U3 C1T 4

Commit message: V4: TPS55288 cryocooler board, 2-pin Pico-Lock on J4
Parts:
- added C10: .1uF, Cryocooler_footprints:GCM21BR72A104KA37L, symbol Device:C
- added C11: 68uF, Cryocooler_footprints:EEH-ZA1V680XP, symbol Device:C
- R4: value 31k -> 30k
- R5: value 2k -> 5k
- R6: value 20k -> 40K
- Rfsw1: value 10k -> 32.4K
Connections:
- net AGND: now also C10.2
- net EN: now also C10.1
- net PGND: now also C11.2
- net at C3.1, C4.1, C5.1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: now also U1.11 (VOUT), C11.1
Other:
- moved on the sheet: J4
