File: Cryocooler_board_4_pin.kicad_pcb (KiCad board)
At the start: 4 copper layers, 58 x 49 mm, 50 parts, among them J1 MOL Pico 4, J2 MOL Pico 4, J3 MOL Pico 4, J4 MOL Pico 2, Q1 IPZ40N04S5-3R1, Q2 IPZ40N04S5-3R1, U1 PTPS55288RPMR, U2 AD5258BRMZ1, U3 C1T 4

Commit message: V4.1 (work in progress): J4 changed to 4-pin Pico-Lock 5040500491
Parts:
- J4: value MOL Pico 2 -> MOL Pico 4; footprint Cryocooler_footprints:MOLEX_2_pin -> Cryocooler_footprints:MOLEX_4_pin
- R6: value 20k -> 40K
- moved J4 0.62 mm to (162.3, 92.9), turned to -90 degrees
Connections:
- J4 pad 2: CRYO_1 -> CRYO_2
- J4 pad 3: (no net) -> CRYO_1
- J4 pad 4: (no net) -> CRYO_1
Routing:
- net CRYO_2: track 48.1 -> 51.0 mm
- net CRYO_1: track 58.8 -> 61.5 mm
