File: Cryocooler_board_4_pin.kicad_sch (KiCad schematic)
At the start: 50 parts, among them J1 MOL Pico 4, J2 MOL Pico 4, J3 MOL Pico 4, J4 MOL Pico 2, Q1 IPZ40N04S5-3R1, Q2 IPZ40N04S5-3R1, U1 PTPS55288RPMR, U2 AD5258BRMZ1, U3 C1T 4

Commit message: V4.1 (work in progress): J4 changed to 4-pin Pico-Lock 5040500491
Parts:
- removed J4: MOL Pico 2, Cryocooler_footprints:MOLEX_2_pin, symbol MOLEX_2_pin:2053380002
- added J4: MOL Pico 4, Cryocooler_footprints:MOLEX_4_pin, symbol MOLEX_4_pin:5040500491
- Cdith1: value 0.047uF -> 15nF
Connections:
- net CRYO_1: now also J4.3
- net CRYO_2: now also J4.1, J4.2
Changed lines of the file:
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@@
 	)
 	(junction
+		(at 231.14 143.51)
+		(diameter 0)
+		(color 0 0 0 0)
+	)
+	(junction
 		(at 100.33 147.32)
 		(diameter 0)
@@
 	(wire
 		(pts
+			(xy 231.14 142.24) (xy 231.14 143.51)
+		)
+		(stroke
+			(width 0)
+			(type default)
+		)
+	)
+	(wire
+		(pts
 			(xy 73.66 92.71) (xy 73.66 95.25)
 		)
@@
 	(wire
 		(pts
+			(xy 231.14 148.59) (xy 231.14 147.32)
+		)
+		(stroke
+			(width 0)
+			(type default)
+		)
+	)
+	(wire
+		(pts
 			(xy 123.19 97.79) (xy 110.49 97.79)
 		)
@@
 	(wire
 		(pts
+			(xy 222.25 148.59) (xy 231.14 148.59)
+		)
+		(stroke
+			(width 0)
+			(type default)
+		)
+	)
+	(wire
+		(pts
 			(xy 92.71 85.09) (xy 110.49 85.09)
 		)
@@
 	(wire
 		(pts
+			(xy 231.14 143.51) (xy 231.14 144.78)
+		)
+		(stroke
+			(width 0)
+			(type default)
+		)
+	)
+	(wire
+		(pts
 			(xy 85.09 157.48) (xy 95.25 157.48)
 		)
@@
 	(wire
 		(pts
+			(xy 222.25 143.51) (xy 231.14 143.51)
+		)
+		(stroke
+			(width 0)
+			(type default)
+		)
+	)
+	(wire
+		(pts
 			(xy 71.12 153.67) (xy 71.12 158.75)
 		)
@@
 	(global_label "CRYO_2"
 		(shape input)
-		(at 227.33 144.78 180)
+		(at 222.25 143.51 180)
 		(fields_autoplaced yes)
 		(effects
@@
 		)
 		(property "Intersheetrefs" "${INTERSHEET_REFS}"
-			(at 217.2086 144.78 0)
+			(at 212.1286 143.51 0)
 			(effects
 				(font
@@
 	(global_label "CRYO_1"
 		(shape input)
-		(at 227.33 147.32 180)
+		(at 222.25 148.59 180)
 		(fields_autoplaced yes)
 		(effects
@@
 		)
 		(property "Intersheetrefs" "${INTERSHEET_REFS}"
-			(at 217.2086 147.32 0)
+			(at 212.1286 148.59 0)
 			(effects
 				(font
@@
 	)
 	(symbol
+		(lib_id "MOLEX_4_pin:5040500491")
+		(at 231.14 142.24 0)
+		(unit 1)
+		(exclude_from_sim no)
+		(in_bom yes)
+		(on_board yes)
+		(dnp no)
+		(property "Reference" "J4"
+			(at 245.364 152.4 90)
+			(effects
+				(font
+					(size 1.524 1.524)
+				)
+				(justify left)
+			)
+		)
+		(property "Value" "MOL Pico 4"
+			(at 247.904 152.654 90)
+			(effects
+				(font
+					(size 1.524 1.524)
+				)
+				(justify left)
+			)
+		)
+		(property "Footprint" "Cryocooler_footprints:MOLEX_4_pin"
+			(at 231.14 142.24 0)
+			(effects
+				(font
+					(size 1.27 1.27)
+					(italic yes)
+				)
+				(hide yes)
+			)
+		)
+		(property "Datasheet" "https://www.molex.com/en-us/products/part-detail-pdf/5040500491?display=pdf"
+			(at 231.14 142.24 0)
+			(effects
+				(font
+					(size 1.27 1.27)
+					(italic yes)
+				)
+				(hide yes)
+			)
+		)
+		(property "Description" ""
+			(at 231.14 142.24 0)
+			(effects
+				(font
+					(size 1.27 1.27)
+				)
+				(hide yes)
+			)
+		)
+		(pin "3"
+		)
+		(pin "2"
+		)
+		(pin "1"
+		)
+		(pin "4"
+		)
+		(instances
+			(project "Cryocooler_board_4_pin"
+				(path "/fc4eef0c-f0fe-4c26-9eed-35cfade9960a"
+					(reference "J4")
+					(unit 1)
+				)
+			)
+		)
+	)
+	(symbol
 		(lib_id "Device:C")
 		(at 102.87 120.65 180)
@@
 			)
 		)
-		(property "Value" "0.047uF"
+		(property "Value" "15nF"
 			(at 112.776 120.904 0)
 			(effects
@@
 					(unit 1)
 				)
-			)
-		)
-	)
-	(symbol
-		(lib_id "MOLEX_2_pin:2053380002")
-		(at 227.33 144.78 0)
-		(unit 1)
-		(exclude_from_sim no)
-		(in_bom yes)
-		(on_board yes)
-		(dnp no)
-		(fields_autoplaced yes)
-		(property "Reference" "J4"
-			(at 241.3 144.7799 0)
-			(effects
-				(font
-					(size 1.524 1.524)
-				)
-				(justify left)
-			)
-		)
-		(property "Value" "MOL Pico 2"
-			(at 241.3 147.3199 0)
-			(effects
-				(font
-					(size 1.524 1.524)
-				)
-				(justify left)
-			)
-		)
-		(property "Footprint" "Cryocooler_footprints:MOLEX_2_pin"
-			(at 227.33 144.78 0)
-			(effects
-				(font
-					(size 1.27 1.27)
-					(italic yes)
-				)
-				(hide yes)
-			)
-		)
-		(property "Datasheet" "https://www.molex.com/en-us/products/part-detail-pdf/2053380002?display=pdf"
-			(at 227.33 144.78 0)
-			(effects
-				(font
-					(size 1.27 1.27)
-					(italic yes)
-				)
-				(hide yes)
-			)
-		)
-		(property "Description" ""
-			(at 227.33 144.78 0)
-			(effects
-				(font
-					(size 1.27 1.27)
-				)
-				(hide yes)
-			)
-		)
-		(pin "2"
-		)
-		(pin "1"
-		)
-		(instances
-			(project ""
-				(path "/fc4eef0c-f0fe-4c26-9eed-35cfade9960a"
-					(reference "J4")
-					(unit 1)
-				)
