File: cryocooler-board.kicad_pcb (KiCad board)
At the start: 4 copper layers, 58 x 49 mm, 50 parts, among them J1 MOL Pico 4, J2 MOL Pico 2, J3 MOL Pico 4, J4 MOL Pico 2, Q1 IPZ40N04S5-3R1, Q2 IPZ40N04S5-3R1, U1 PTPS55288RPMR, U2 AD5258BRMZ1, U3 C1T 4

Commit message: V4.1 as ordered: loop-stability test build
- Values: Cp1 100 pF C0G, Cc1 C0G, R6 41.2k (8 A), R5 5.1k, Cdith1 15 nF
- Added C12 (ISP-ISN filter), R9 (DNP dither disable), TP_COMP1, TP_VCC1
- R7 moved next to Q1 gate; passives on standard IPC footprints
- MF/MP/LCSC fields on all parts; ERC fixes (PWR_FLAGs, pin types)
- Production files regenerated (Fabrication Toolkit)
- README updated; new 3D, layer and Bode images (12 V and 20 V)
Parts:
- added C12: 0.1uF, Capacitor_SMD:C_0603_1608Metric, F.Cu at (158.9, 86.1)
- added R9: 0 Ohm, Resistor_SMD:R_0603_1608Metric, F.Cu at (148.9, 95.0)
- added TP_COMP1: TestPoint, TestPoint:TestPoint_THTPad_D1.5mm_Drill0.7mm, F.Cu at (144.5, 76.5)
- added TP_VCC1: TestPoint, TestPoint:TestPoint_THTPad_D1.5mm_Drill0.7mm, F.Cu at (134.4, 70.2)
- C1, C2, C9: footprint Cryocooler:GCM21BR72A104KA37L -> Capacitor_SMD:C_0805_2012Metric
- C10: value .1uF -> 0.1uF; footprint Cryocooler:GCM21BR72A104KA37L -> Capacitor_SMD:C_0805_2012Metric
- C3, C4, C5, C6, CIN1, CIN2: footprint Cryocooler:CGA5L1X7R1H106K160AC -> Capacitor_SMD:C_1206_3216Metric
- C7, C8, CIN4: footprint Cryocooler:CGA3E3X5R1H105M080AB -> Capacitor_SMD:C_0603_1608Metric
- CVCC1: footprint Cryocooler:GRT188R61C475KE13D -> Capacitor_SMD:C_0603_1608Metric
- Cc1: footprint Cryocooler:CGA3E2C0G1H562J080AA -> Capacitor_SMD:C_0603_1608Metric
- Cdith1: footprint Cryocooler:CGA3E2X7R1H473K080AD -> Capacitor_SMD:C_0603_1608Metric
- Cp1: value 22pF -> 100pF; footprint Cryocooler:CGA3E2NP01H220J080AA -> Capacitor_SMD:C_0603_1608Metric
- Q1, Q2: value IPZ40N04S5-3R1 -> IPZ40N04S5L4R8ATMA1
- R1, R2: footprint Cryocooler:CRCW12062K20JNEA -> Resistor_SMD:R_1206_3216Metric
- R3: value 10mili Ohms -> 10mOhm; footprint Cryocooler:CRF1206-FZ-R010ELF -> Resistor_SMD:R_1206_3216Metric
- R4: footprint Cryocooler:CRCW080530K9FKEA -> Resistor_SMD:R_0805_2012Metric
- R5: value 5k -> 5.1k; footprint Cryocooler:CRCW08052K00FKEA -> Resistor_SMD:R_0805_2012Metric
- R6: value 40K -> 41.2K; footprint Cryocooler:CRCW120620K0FKEAC -> Resistor_SMD:R_1206_3216Metric
- R7, R8: footprint Cryocooler:CRCW08051R00JNEAHP -> Resistor_SMD:R_0805_2012Metric
- Rc1: footprint Cryocooler:CRCW060326K1FKEA -> Resistor_SMD:R_0603_1608Metric
- Rfsw1: footprint Cryocooler:CRCW060310K0FKEA -> Resistor_SMD:R_0603_1608Metric
- U1: value PTPS55288RPMR -> TPS55288RPMR
- U3: value C1T 4 -> 4A Fuse
- moved R7 13.5 mm to (131.6, 93.1), turned to 180 degrees
- moved C10 1.26 mm to (128.1, 79.2)
- moved R5 1.26 mm to (126.0, 79.2)
- moved L1 1.17 mm to (135.2, 86.4)
- moved Rfsw1 0.10 mm to (149.7, 91.4)
- moved Cdith1 0.10 mm to (148.2, 91.5)
- moved R6 0.07 mm to (148.1, 80.3)
Routing:
- net Net-(Q1-G): track 20.5 -> 1.79 mm, vias 2 -> 0
- net Net-(U1-DR1H): track 8.83 -> 23.1 mm, vias 0 -> 2
- net Net-(U1-COMP): track 5.63 -> 14.4 mm, vias 0 -> 2
- net Net-(U1-DITH/SYNC): track 2.31 -> 7.72 mm
- net VCC: track 29.2 -> 34.3 mm
- net AGND: track 51.1 -> 53.4 mm
- net PGND: track 3.10 -> 4.05 mm, vias 115 -> 117
- net /EN: track 35.9 -> 35.3 mm
Other:
- board text added: "->"
- board text added: "COMP"
- board text added: "Cryocooler Board V4.1 Rodrigo Spinola e Castro"
- board text added: "Dither Switch"
- board text added: "Local I2C Power, 2.2Kohm"
- board text added: "SW1"
- board text added: "VCC"
- board text removed: "Cryocooler Board V4 Rodrigo Spinola e Castro"
