File: cryocooler-board.kicad_sch (KiCad schematic)
At the start: 50 parts, among them J1 MOL Pico 4, J2 MOL Pico 2, J3 MOL Pico 4, J4 MOL Pico 2, Q1 IPZ40N04S5-3R1, Q2 IPZ40N04S5-3R1, U1 PTPS55288RPMR, U2 AD5258BRMZ1, U3 C1T 4

Commit message: V4.1 as ordered: loop-stability test build
- Values: Cp1 100 pF C0G, Cc1 C0G, R6 41.2k (8 A), R5 5.1k, Cdith1 15 nF
- Added C12 (ISP-ISN filter), R9 (DNP dither disable), TP_COMP1, TP_VCC1
- R7 moved next to Q1 gate; passives on standard IPC footprints
- MF/MP/LCSC fields on all parts; ERC fixes (PWR_FLAGs, pin types)
- Production files regenerated (Fabrication Toolkit)
- README updated; new 3D, layer and Bode images (12 V and 20 V)
Parts:
- added C12: 0.1uF, Capacitor_SMD:C_0603_1608Metric, symbol Device:C
- added R9: 0 Ohm, Resistor_SMD:R_0603_1608Metric, symbol Device:R_US
- added TP_COMP1, TP_VCC1: TestPoint, TestPoint:TestPoint_THTPad_D1.5mm_Drill0.7mm, symbol Connector:TestPoint
- C1, C2, C9: footprint Cryocooler:GCM21BR72A104KA37L -> Capacitor_SMD:C_0805_2012Metric; LCSC Part # (none) -> C85866; MF (none) -> Murata; MP (none) -> GCM21BR72A104KA37L
- C10: value .1uF -> 0.1uF; footprint Cryocooler:GCM21BR72A104KA37L -> Capacitor_SMD:C_0805_2012Metric; LCSC Part # (none) -> C85866; MF (none) -> Murata; MP (none) -> GCM21BR72A104KA37L
- C11, CIN3: LCSC Part # (none) -> C242137; MF (none) -> Panasonic; MP (none) -> EEH-ZA1V680XP
- C3, C4, C5, C6, CIN1, CIN2: footprint Cryocooler:CGA5L1X7R1H106K160AC -> Capacitor_SMD:C_1206_3216Metric; LCSC Part # (none) -> C13585; MF (none) -> Samsung; MP (none) -> CL31A106KBHNNNE
- C7, C8, CIN4: footprint Cryocooler:CGA3E3X5R1H105M080AB -> Capacitor_SMD:C_0603_1608Metric; LCSC Part # (none) -> C49326360; MF (none) -> AIDE; MP (none) -> 0603X5R105K500NT
- CVCC1: footprint Cryocooler:GRT188R61C475KE13D -> Capacitor_SMD:C_0603_1608Metric; LCSC Part # (none) -> C437574; MF (none) -> Murata; MP (none) -> GRT188R61C475KE13D
- Cc1: footprint Cryocooler:CGA3E2C0G1H562J080AA -> Capacitor_SMD:C_0603_1608Metric; LCSC Part # (none) -> C440183; MF (none) -> Murata; MP (none) -> GRM1885C1H562JA01D
- Cdith1: footprint Cryocooler:CGA3E2X7R1H473K080AD -> Capacitor_SMD:C_0603_1608Metric; LCSC Part # (none) -> C2180652; MF (none) -> TDK; MP (none) -> CGA3E2X7R1H153K080AA
- Cp1: value 22pF -> 100pF; footprint Cryocooler:CGA3E2NP01H220J080AA -> Capacitor_SMD:C_0603_1608Metric; LCSC Part # (none) -> C71664; MF (none) -> Murata; MP (none) -> GRM1885C1H101JA01D
- J1, J3: LCSC Part # (none) -> C177235; MF (none) -> Molex; MP (none) -> 5040500491
- J2, J4: LCSC Part # (none) -> C17575002; MF (none) -> Molex; MP (none) -> 2053380002
- L1: MP (none) -> XAL1010-103MED
- Q1, Q2: value IPZ40N04S5-3R1 -> IPZ40N04S5L4R8ATMA1; symbol Cryocooler:IPZ40N04S5-3R1 -> Cryocooler:IPZ40N04S5L4R8ATMA1; Availability In Stock -> (none); Check_prices https://www.snapeda.com/parts/IPZ40N04S5-3R1/Infineon/view-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 -> (none); Description_1 MOSFET, AEC-Q101, N-CH, 40V, TSDSON; Transistor Polarity:N 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 -> (none); LCSC Part # (none) -> C6969335; MF Infineon Technologies -> Infineon; MP IPZ40N04S5-3R1 -> IPZ40N04S5L4R8ATMA1; Package None -> (none); Price None -> (none); SnapEDA_Link https://www.snapeda.com/parts/IPZ40N04S5-3R1/Infineon/view-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 -> (none)
- R1, R2: footprint Cryocooler:CRCW12062K20JNEA -> Resistor_SMD:R_1206_3216Metric; LCSC Part # (none) -> C6538126; MF (none) -> Vishay; MP (none) -> CRCW12062K20JNEA
- R3: value 10mili Ohms -> 10mOhm; footprint Cryocooler:CRF1206-FZ-R010ELF -> Resistor_SMD:R_1206_3216Metric; LCSC Part # (none) -> C5629523; MF (none) -> Bourns; MP (none) -> CRF1206-FZ-R010ELF
- R4: footprint Cryocooler:CRCW080530K9FKEA -> Resistor_SMD:R_0805_2012Metric; LCSC Part # (none) -> C844838; MF (none) -> Vishay; MP (none) -> CRCW080530K0FKEA
- R5: value 5k -> 5.1k; footprint Cryocooler:CRCW08052K00FKEA -> Resistor_SMD:R_0805_2012Metric; LCSC Part # (none) -> C844854; MF (none) -> Vishay; MP (none) -> CRCW08055K10FKEA
- R6: value 40K -> 41.2K; footprint Cryocooler:CRCW120620K0FKEAC -> Resistor_SMD:R_1206_3216Metric; LCSC Part # (none) -> C3017228; MF (none) -> VO; MP (none) -> SCR1206F41K2
- R7, R8: footprint Cryocooler:CRCW08051R00JNEAHP -> Resistor_SMD:R_0805_2012Metric; LCSC Part # (none) -> C2078379; MF (none) -> Vishay; MP (none) -> CRCW08051R00JNEAHP
- Rc1: footprint Cryocooler:CRCW060326K1FKEA -> Resistor_SMD:R_0603_1608Metric; LCSC Part # (none) -> C844150; MF (none) -> Vishay; MP (none) -> CRCW060326K1FKEA
- Rfsw1: footprint Cryocooler:CRCW060310K0FKEA -> Resistor_SMD:R_0603_1608Metric; LCSC Part # (none) -> C844154; MF (none) -> Vishay; MP (none) -> CRCW060332K4FKEA
- U1: value PTPS55288RPMR -> TPS55288RPMR; LCSC Part # (none) -> C2864583; MF (none) -> Texas Instruments; MP (none) -> TPS55288RPMR
- U2: LCSC Part # (none) -> C649444; MF (none) -> Analog Devices; MP (none) -> AD5258BRMZ1
- U3: value C1T 4 -> 4A Fuse; LCSC Part # (none) -> C2838918; MF (none) -> prosemi; MP (none) -> 1206TD-4A
Connections:
- net AGND: now also R9.2
- net VCC: now also TP_VCC1.1
- net VOUT: now also C12.2
- net at Cp1.1, Rc1.2, U1.18 (COMP): now also TP_COMP1.1
- net at Cdith1.2, U1.7 (DITH/SYNC): now also R9.1
- net at C11.1, C3.1, C4.1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: now also C12.1
